File: ice-dongle.kicad_sch (KiCad schematic)
At the start: 43 parts, among them J1 USB4155-03-C_REVA, J2 NC Jumper, J3 PROG HEADER, J4 FFC2B35-18-G_REVA2, SW1 SW_Push, SW2 SW_Push, U1 APS6404L-3SQR, U2 W25Q64JWUUIQ, U3 DRTR5V0U4S, U4 MCP1824x-OT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

Commit message: USB-C jack, finish layout
Parts:
- removed J1: USB4155-03-C_REVA, emeb_library:GCT_USB4155-03-C_REVA, symbol emeb_library:USB4155-03-C_REVA
- added J1: USB_C_Receptacle_USB2.0, Connector_USB:USB_C_Receptacle_HRO_TYPE-C-31-M-12, symbol Connector:USB_C_Receptacle_USB2.0
- J3: footprint Connector_PinHeader_1.27mm:PinHeader_2x04_P1.27mm_Vertical_SMD -> Connector_PinHeader_1.27mm:PinHeader_2x05_P1.27mm_Vertical_SMD; symbol Connector_Generic:Conn_02x04_Odd_Even -> Connector_Generic:Conn_02x05_Odd_Even
Connections:
- net ES_BKL: now also U6.44 (IOB_3b_G6); no longer U6.48 (IOB_4a)
- net ES_DC: now also U6.48 (IOB_4a); no longer U6.44 (IOB_3b_G6)
- net ES_P11: now also U6.25 (IOT_36b); no longer U6.32 (IOT_43a)
- net ES_P12: now also U6.26 (IOT_39a); no longer U6.31 (IOT_42b)
- net ES_P13: now also U6.27 (IOT_38b); no longer U6.28 (IOT_41a)
- net ES_P14: now also U6.28 (IOT_41a); no longer U6.27 (IOT_38b)
- net ES_P15: now also U6.31 (IOT_42b); no longer U6.26 (IOT_39a)
- net ES_P16: now also U6.32 (IOT_43a); no longer U6.25 (IOT_36b)
- net ES_P17: now also U6.34 (IOT_44b); no longer U6.23 (IOT_37a)
- net ES_P18: now also U6.36 (IOT_48b); no longer U6.21 (IOB_23b)
- net ES_POCI: now also U6.47 (IOB_2a); no longer U6.45 (IOB_5a)
- net ES_RST: now also U6.20 (IOB_25b_G3); no longer U6.43 (IOT_49a)
- net ES_SCK: now also U6.45 (IOB_5a); no longer U6.47 (IOB_2a)
- net ES_SDCS: now also U6.23 (IOT_37a); no longer U6.34 (IOT_44b)
- net ES_TFTCS: now also U6.21 (IOB_23b); no longer U6.36 (IOT_48b)
- net GND: now also R1.1, R6.1, J1.A1 (GND), J1.A12 (GND), J1.B1 (GND), J1.B12 (GND); no longer R1.2, R6.2
- net VUSB: now also J1.A4 (VBUS), J1.A9 (VBUS), J1.B4 (VBUS), J1.B9 (VBUS)
- net SPARE10: now reaches U6.11 (IOB_20a)
- net SPARE10: now also J3.10 (Pin_10)
- net SPARE9: now reaches U6.12 (IOB_22A)
- net SPARE9: now also J3.9 (Pin_9)
- net at R7.2, R8.2, U3.4: now also J1.A6 (D+), J1.B6 (D+)
- net at R9.2, U3.6: now also J1.A7 (D-), J1.B7 (D-)
- net at R5.2: now also J1.B5 (CC2)
- net +3V3 renamed +3.3V
- new net: J1.S1 (SHIELD), R6.2
- new net: J1.A5 (CC1), R1.2
- no-connect marks 20 -> 9
Other:
- note added: "vcc"
- moved on the sheet: R1, R5, R6

Commit message: Fix Eye-SPI pinout, add VIN selector
Parts:
- added JP1: Jumper_3_Bridged12, Jumper:SolderJumper-3_P1.3mm_Bridged12_RoundedPad1.0x1.5mm, symbol Jumper:Jumper_3_Bridged12
- U4: symbol ice-dongle-rescue:MCP1824x-OT-emeb_library -> emeb_library:MCP1824x-OT
- U6: symbol ice-dongle-rescue:ice5lp4k_sg48-emeb_library -> emeb_library:ice5lp4k_sg48
Connections:
- net +3.3V: now also JP1.1 (A); no longer J4.1
- net ES_BKL: now also J4.17, U6.36 (IOT_48b); no longer J4.2, U6.44 (IOB_3b_G6)
- net ES_DC: now also J4.12, U6.28 (IOT_41a); no longer J4.7, U6.48 (IOB_4a)
- net ES_PICO: now also J4.14, U6.32 (IOT_43a); no longer J4.5, U6.46 (IOB_0a)
- net ES_POCI: now also J4.13, U6.31 (IOT_42b); no longer J4.6, U6.47 (IOB_2a)
- net ES_RST: now also J4.11, U6.27 (IOT_38b); no longer J4.8, U6.20 (IOB_25b_G3)
- net ES_SCK: now also J4.15, U6.34 (IOT_44b); no longer J4.4, U6.45 (IOB_5a)
- net ES_SDCS: now also J4.9, U6.25 (IOT_36b); no longer J4.10, U6.23 (IOT_37a)
- net ES_TFTCS: now also J4.10, U6.26 (IOT_39a); no longer J4.9, U6.21 (IOB_23b)
- net GND: now also J4.16; no longer J4.3
- net VUSB: now also JP1.3 (B)
- removed net ES_P11: J4.11, U6.25 (IOT_36b)
- removed net ES_P12: J4.12, U6.26 (IOT_39a)
- removed net ES_P13: J4.13, U6.27 (IOT_38b)
- removed net ES_P14: J4.14, U6.28 (IOT_41a)
- removed net ES_P15: J4.15, U6.31 (IOT_42b)
- removed net ES_P16: J4.16, U6.32 (IOT_43a)
- removed net ES_P17: J4.17, U6.34 (IOT_44b)
- net ES_P18 renamed ES_VIN
- net ES_VIN: now also JP1.2 (C); no longer U6.36 (IOT_48b)
- new net ES_BUSY: J4.3, U6.46 (IOB_0a)
- new net ES_GP1: J4.2, U6.45 (IOB_5a)
- new net ES_GP2: J4.1, U6.44 (IOB_3b_G6)
- new net ES_INT: J4.4, U6.47 (IOB_2a)
- new net ES_MEMCS: J4.8, U6.23 (IOT_37a)
- new net ES_SCL: J4.6, U6.20 (IOB_25b_G3)
- new net ES_SDA: J4.5, U6.48 (IOB_4a)
- new net ES_TSCS: J4.7, U6.21 (IOB_23b)
- no-connect marks 9 -> 10
Other:
- note added: "NOTE: Pin numbering of this symbol is reversed from that used by Adafruit"
- note added: "Select VIN source"

Commit message: Clean up USB & RGB routing.
Other:
- note added: "Pin 37 (USB_PU) is output-only when pin 35 is used as PLL pad input."
Changed lines of the file:
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@@
     (effects (font (size 1.524 1.524)) (justify right bottom))
+  )
+  (text "Pin 37 (USB_PU) is output-only\nwhen pin 35 is used as PLL pad input."
+    (at 322.58 46.99 0)
+    (effects (font (size 1.27 1.27)) (justify left bottom))
   )
   (text "NOTE: Pin numbering of this symbol\nis reversed from that used by\nAdafruit "

Commit message: Added
Parts:
- added J5: Qwiic, Connector_PinHeader_1.27mm:PinHeader_1x04_P1.27mm_Vertical, symbol Connector_Generic:Conn_01x04
Connections:
- net +3.3V: now also J5.2 (Pin_2)
- net GND: now also J5.1 (Pin_1)
- net at U6.3 (IOB_9b): now also J5.4 (Pin_4)
- net at U6.43 (IOT_49a): now also J5.3 (Pin_3)
- no-connect marks 10 -> 8
Other:
- note added: "Blk - GND"
- note added: "Blu - SDA"
- note added: "Red - 3v3"
- note added: "Yel - SCL"
Changed lines of the file:
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@@
   (no_connect (at 271.78 72.39))
   (no_connect (at 288.29 110.49))
-  (no_connect (at 271.78 69.85))
   (no_connect (at 271.78 87.63))
   (no_connect (at 271.78 85.09))
   (no_connect (at 139.7 62.23))
-  (no_connect (at 300.99 49.53))
   (wire (pts (xy 110.49 137.16) (xy 121.92 137.16))
     (stroke (width 0) (type default) (color 0 0 0 0))
@@
     (stroke (width 0) (type default) (color 0 0 0 0))
   )
+  (wire (pts (xy 262.89 39.37) (xy 243.84 39.37))
+    (stroke (width 0) (type default) (color 0 0 0 0))
+  )
   (wire (pts (xy 229.87 208.28) (xy 223.52 208.28))
     (stroke (width 0) (type default) (color 0 0 0 0))
@@
     (stroke (width 0) (type default) (color 0 0 0 0))
   )
+  (wire (pts (xy 247.65 22.86) (xy 247.65 27.94))
+    (stroke (width 0) (type default) (color 0 0 0 0))
+  )
   (wire (pts (xy 407.67 54.61) (xy 407.67 67.31))
     (stroke (width 0) (type default) (color 0 0 0 0))
@@
     (stroke (width 0) (type default) (color 0 0 0 0))
   )
+  (wire (pts (xy 271.78 69.85) (xy 262.89 69.85))
+    (stroke (width 0) (type default) (color 0 0 0 0))
+  )
   (wire (pts (xy 106.68 38.1) (xy 106.68 43.18))
     (stroke (width 0) (type default) (color 0 0 0 0))
@@
     (stroke (width 0) (type default) (color 0 0 0 0))
   )
+  (wire (pts (xy 300.99 36.83) (xy 300.99 49.53))
+    (stroke (width 0) (type default) (color 0 0 0 0))
+  )
   (wire (pts (xy 345.44 85.09) (xy 349.25 85.09))
     (stroke (width 0) (type default) (color 0 0 0 0))
@@
     (stroke (width 0) (type default) (color 0 0 0 0))
   )
+  (wire (pts (xy 243.84 34.29) (xy 254 34.29))
+    (stroke (width 0) (type default) (color 0 0 0 0))
+  )
   (wire (pts (xy 401.32 53.34) (xy 401.32 40.64))
     (stroke (width 0) (type default) (color 0 0 0 0))
@@
     (stroke (width 0) (type default) (color 0 0 0 0))
   )
+  (wire (pts (xy 243.84 36.83) (xy 300.99 36.83))
+    (stroke (width 0) (type default) (color 0 0 0 0))
+  )
   (wire (pts (xy 110.49 107.95) (xy 121.92 107.95))
     (stroke (width 0) (type default) (color 0 0 0 0))
@@
     (stroke (width 0) (type default) (color 0 0 0 0))
   )
+  (wire (pts (xy 262.89 69.85) (xy 262.89 39.37))
+    (stroke (width 0) (type default) (color 0 0 0 0))
+  )
   (wire (pts (xy 407.67 40.64) (xy 407.67 49.53))
     (stroke (width 0) (type default) (color 0 0 0 0))
@@
     (stroke (width 0) (type default) (color 0 0 0 0))
   )
+  (wire (pts (xy 243.84 22.86) (xy 247.65 22.86))
+    (stroke (width 0) (type default) (color 0 0 0 0))
+  )
   (wire (pts (xy 306.07 24.13) (xy 311.15 24.13))
     (stroke (width 0) (type default) (color 0 0 0 0))
@@
     (stroke (width 0) (type default) (color 0 0 0 0))
   )
+  (wire (pts (xy 243.84 31.75) (xy 243.84 22.86))
+    (stroke (width 0) (type default) (color 0 0 0 0))
+  )
   (wire (pts (xy 74.93 105.41) (xy 74.93 139.7))
     (stroke (width 0) (type default) (color 0 0 0 0))
@@
     (effects (font (size 1.524 1.524)) (justify right bottom))
   )
+  (text "Yel - SCL" (at 226.06 40.64 0)
+    (effects (font (size 1.27 1.27)) (justify left bottom))
+  )
   (text "RST" (at 181.61 114.3 0)
     (effects (font (size 1.524 1.524)) (justify left bottom))
   )
+  (text "Blk - GND" (at 226.06 33.02 0)
+    (effects (font (size 1.27 1.27)) (justify left bottom))
+  )
   (text "USR Button" (at 146.05 114.3 0)
     (effects (font (size 1.524 1.524)) (justify left bottom))
+  )
+  (text "Red - 3v3" (at 226.06 35.56 0)
+    (effects (font (size 1.27 1.27)) (justify left bottom))
   )
   (text "Note: SO/SI lines swap direction depending on which device is being loaded.\nFPGA - SO = Output from Prog to FPGA, SI = Input from FPGA to Prog\nFlash - SO = Input from Flash to Prog, SI = Output from Prog to Flash"
@@
   (text "NOTE: Pin numbering of this symbol\nis reversed from that used by\nAdafruit "
     (at 365.76 204.47 0)
+    (effects (font (size 1.27 1.27)) (justify left bottom))
+  )
+  (text "Blu - SDA" (at 226.06 38.1 0)
     (effects (font (size 1.27 1.27)) (justify left bottom))
   )
@@
     (pin "9")
   )
+  (symbol (lib_id "Connector_Generic:Conn_01x04") (at 238.76 34.29 0) (mirror y) (unit 1)
+    (in_bom yes) (on_board yes) (fields_autoplaced)
+    (property "Reference" "J5" (id 0) (at 238.76 25.4 0))
+    (property "Value" "Qwiic" (id 1) (at 238.76 27.94 0))
+    (property "Footprint" "Connector_PinHeader_1.27mm:PinHeader_1x04_P1.27mm_Vertical" (id 2) (at 238.76 34.29 0)
+      (effects (font (size 1.27 1.27)) hide)
+    )
+    (property "Datasheet" "~" (id 3) (at 238.76 34.29 0)
+      (effects (font (size 1.27 1.27)) hide)
+    )
+    (pin "1")
+    (pin "2")
+    (pin "3")
+    (pin "4")
+  )
   (symbol (lib_id "Jumper:Jumper_3_Bridged12") (at 360.68 138.43 0) (unit 1)
     (in_bom yes) (on_board yes) (fields_autoplaced)
@@
     (pin "2")
   )
+  (symbol (lib_id "power:GND") (at 247.65 27.94 0) (unit 1)
+    (in_bom yes) (on_board yes)
+    (property "Reference" "#PWR042" (id 0) (at 247.65 34.29 0)
+      (effects (font (size 1.27 1.27)) hide)
+    )
+    (property "Value" "GND" (id 1) (at 247.65 31.75 0))
+    (property "Footprint" "" (id 2) (at 247.65 27.94 0))
+    (property "Datasheet" "" (id 3) (at 247.65 27.94 0))
+    (pin "1")
+  )
+  (symbol (lib_id "power:+3.3V") (at 254 34.29 0) (unit 1)
+    (in_bom yes) (on_board yes)
+    (property "Reference" "#PWR041" (id 0) (at 254 38.1 0)
+      (effects (font (size 1.27 1.27)) hide)
+    )
+    (property "Value" "+3.3V" (id 1) (at 254 30.734 0))
+    (property "Footprint" "" (id 2) (at 254 34.29 0)
+      (effects (font (size 1.27 1.27)) hide)
+    )
+    (property "Datasheet" "" (id 3) (at 254 34.29 0)
+      (effects (font (size 1.27 1.27)) hide)
+    )
+    (pin "1")
+  )
   (symbol (lib_id "Device:R") (at 100.33 38.1 270) (unit 1)
     (in_bom yes) (on_board yes)
@@
       (reference "#PWR040") (unit 1) (value "GND") (footprint "")
     )
+    (path "/cd4af5b2-d58f-49a2-9d53-7a62c610baea"
+      (reference "#PWR041") (unit 1) (value "+3.3V") (footprint "")
+    )
+    (path "/cc36456c-b381-4041-9f4b-5288a1568589"
+      (reference "#PWR042") (unit 1) (value "GND") (footprint "")
+    )
     (path "/00000000-0000-0000-0000-00005fcfe6ed"
       (reference "C1") (unit 1) (value "0.1uf") (footprint "Capacitor_SMD:C_0402_1005Metric")
@@
       (reference "J4") (unit 1) (value "FFC2B35-18-G_REVA2") (footprint "emeb_library:GCT_FFC2B35-18-G_REVA2")
     )
+    (path "/3b18ab27-0612-4b95-838f-57721f9e8525"
+      (reference "J5") (unit 1) (value "Qwiic") (footprint "Connector_PinHeader_1.27mm:PinHeader_1x04_P1.27mm_Vertical")
+    )
     (path "/447ddc46-d902-4be2-9016-1798cc2d72f2"

Commit message: Minor cleanups, add unmarked testpoints to unused IO
Parts:
- added TP1, TP2: TestPoint, emeb_library:TestPoint_Pad_D0.5mm, symbol Connector:TestPoint
Connections:
- net +3.3V: now also JP1.3 (B); no longer JP1.1 (A)
- net VUSB: now also JP1.1 (A); no longer JP1.3 (B)
- net at U6.10 (IOB_18a): now also TP2.1
- net at U6.9 (IOB_16a): now also TP1.1
- no-connect marks 8 -> 6
